File: hw/teamc-carrier/radio.kicad_sch (KiCad schematic)
At the start: 10 parts, among them U7 E01-ML01SP4

Commit message: carrier: review fixes (Si2333DDS, BCM857BS, fuse, soft start, D_SMF, pull-ups to 3V3_PI, MODE->VIN), power+SPI routed (DRC 0 errors), GND vias, BoM, design notes; CLAUDE.md session log
Co-Authored-By: Claude Opus 5.5 <noreply@anthropic.com>
Claude-Session: https://claude.ai/code/session_01Dy4TuRNF8V28KreA3jwCtM
Connections:
- net 3V3_RADIO: no longer R80.1, R81.1
- new net 3V3_PI: R80.1, R81.1
Other:
- note added: "PULL-UPS TO 3V3_PI"
- note removed: "PULL-UPS TO 3V3_RADIO"
Changed lines of the file:
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@@
 		)
 	)
-	(global_label "3V3_RADIO"
+	(global_label "3V3_PI"
 		(shape passive)
 		(at 57.15 190.5 180)
@@
 		)
 	)
-	(global_label "3V3_RADIO"
+	(global_label "3V3_PI"
 		(shape passive)
 		(at 57.15 208.28 180)
@@
 		)
 	)
-	(text "PULL-UPS TO 3V3_RADIO"
+	(text "PULL-UPS TO 3V3_PI"
 		(exclude_from_sim no)
 		(at 25.4 172.72 0)
