File: hw/teamc-carrier/power.kicad_sch (KiCad schematic)
At the start: 58 parts, among them J2 USB-C charge, J20 BATT 18650, J21 BATT 2 (DNP), J22 PWR toggle, Q1 AO3401A, Q2 AO3401A, Q3 2N7002, Q4 AO3401A, U1 MCP73831, U12 SP0504BAHTG, U2 TPS61022, U3 BC857BS, U4 TLV75533, U5 TPS63001, U6 MAX17048

Commit message: carrier: review fixes (Si2333DDS, BCM857BS, fuse, soft start, D_SMF, pull-ups to 3V3_PI, MODE->VIN), power+SPI routed (DRC 0 errors), GND vias, BoM, design notes; CLAUDE.md session log
Co-Authored-By: Claude Opus 5.5 <noreply@anthropic.com>
Claude-Session: https://claude.ai/code/session_01Dy4TuRNF8V28KreA3jwCtM
Parts:
- added C18: 100n 50V X7R, Capacitor_SMD:C_0805_2012Metric_Pad1.18x1.45mm_HandSolder, symbol Device:C
- added F1: 5A fast, Fuse:Fuse_1206_3216Metric_Pad1.42x1.75mm_HandSolder, symbol Device:Fuse
- D1, D2, D3: footprint Diode_SMD:D_SOD-123F -> Diode_SMD:D_SMF
- Q1, Q2: value AO3401A -> Si2333DDS; MPN AO3401A -> Si2333DDS-T1-GE3; Manufacturer Alpha & Omega -> Vishay
- R9: value 1k 1% -> 10k 1%; MPN RC0805FR-071KL -> RC0805FR-0710KL
- U3: value BC857BS -> BCM857BS; MPN BC857BS,115 -> BCM857BS,115
Connections:
- net BAT_RAW: now also F1.2; no longer J20.1 (Pin_1), J21.1 (Pin_1)
- net GND: no longer U2.6 (MODE)
- net PWR_G: now also C18.1
- net VBAT: now also C18.2
- net VBAT_SW: now also U2.6 (MODE)
- new net BAT_IN: F1.1, J20.1 (Pin_1), J21.1 (Pin_1)
Other:
- note added: "Toggle (E-Switch 100SP1T1B1M1QEH, off-board), closed = ON: pulls PWR_G low through R9 (10 k; C18 makes a ~1 ms soft start) → Q2 on. Open: R8 holds Q2 off and its body diode blocks VBAT → VBAT_SW. The toggle carries ~40 µA only. ESD on PWR_SW_J: U12 pin 4."
- note added: "VDD/CELL: Kelvin trace from Q1's source (VBAT), GND to J20, not along the boost input path; it reads the cell ~I x RDS(Q1) low under load (safe side for the thresholds). No I2C pull-ups here (the Pi has 1.8 k). Software: never set MODE.EnSleep."
- note added: "VOUT = 0.600 V x (1 + 750k/100k) = 5.10 V (PFM 5.15 V; OVP 5.5 V min). L1 744316100 is in TI's Table 8-2; peak ~5.7 A at 3.0 V in / 2.5 A out. C3 100 pF: feed-forward zero 1/(2π·750k·100p) = 2.1 kHz (§8.2.2.4, COUT_eff > 40 µF). EN = VBAT_SW: on with the switch. MODE = VIN: forced PWM (layout, 19-Oct: MODE sits between VIN and EN, so it shares their copper; PFM would only save a few mA below ~100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"
- note removed: "Toggle (E-Switch 100SP1T1B1M1QEH, off-board), closed = ON: pulls PWR_G low through R9 → Q2 on. Open: R8 holds Q2 off and its body diode blocks VBAT → VBAT_SW. The toggle carries ~40 µA only. ESD on PWR_SW_J: U12 pin 4."
- note removed: "VDD/CELL and GND: Kelvin traces to J20, not along the boost input path. No I2C pull-ups here (the Pi has 1.8 k). Software: never set MODE.EnSleep."
- note removed: "VOUT = 0.600 V x (1 + 750k/100k) = 5.10 V (PFM 5.15 V; OVP 5.5 V min). L1 744316100 is in TI's Table 8-2; peak ~5.7 A at 3.0 V in / 2.5 A out. C3 100 pF: feed-forward zero 1/(2π·750k·100p) = 2.1 kHz (§8.2.2.4, COUT_eff > 40 µF). EN = VBAT_SW: on with the switch. MODE = GND: auto PFM (light-load efficiency, no reverse inductor current). C5 bulk: the cell sits on a lead (§8.2.2.5). Tight SW loop, V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"

Commit message: carrier: re-placed in clusters, boost GND pocket fixed, SP4 keep-out on both layers, power+SPI routed (DRC 0 errors); small nets handed to ET; JLCPCB-class 0.2 mm rules
- removed SW1 (bench button), J21 (2nd cell -> harness), D1 (VBUS ESD on U12's spare channel)
- router: rip-up/reroute + negotiated congestion options (neither finished the small nets at 0.3 mm)
- design notes: hand-off list for ET, fab rules, layout-driven changes; BoM ~EUR 102/device

Co-Authored-By: Claude Opus 5.5 <noreply@anthropic.com>
Claude-Session: https://claude.ai/code/session_01Dy4TuRNF8V28KreA3jwCtM
Parts:
- removed D1: SMF5.0A, Diode_SMD:D_SMF, symbol Diode:SMF5V0A
- removed J21: BATT 2 (DNP), Connector_JST:JST_VH_B2P-VH_1x02_P3.96mm_Vertical, symbol Connector_Generic:Conn_01x02
Connections:
- net VBUS_USB: now also U12.5 (K)
- no-connect marks 1 -> 0
Other:
- note added: "Cells: protected 18650 (PCM inside) in an MPD BH-18650-PC holder on the box floor (off-board), lead to J20 (JST-VH, 10 A). 2nd cell: a 2nd holder wired in parallel into the same J20 lead (harness; matched cells only). Q1: the body diode conducts for a correct cell, then VGS = -VBAT turns it on; a reversed cell is blocked. D3: ESD/hot-plug clamp. Do not plug USB with a reversed cell (the charger, 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"
- note removed: "Cells: protected 18650 (PCM inside) in an MPD BH-18650-PC holder on the box floor (off-board), lead to J20 (JST-VH, 10 A). J21 = second cell in parallel (DNP; only matched cells). Q1: the body diode conducts for a correct cell, then VGS = -VBAT turns it on; a reversed cell is blocked. D3: ESD/hot-plug clamp. Do not plug USB with a reversed cell (the charger, current-limited, would bias Q1 partly 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"
