File: hw/teamc-carrier/ui.kicad_sch (KiCad schematic)
At the start: 21 parts, among them J10 GO/STOP button, J11 role toggle, J12 mode toggle, SW1 bench GO/STOP, U11 SP0504BAHTG

Commit message: carrier: re-placed in clusters, boost GND pocket fixed, SP4 keep-out on both layers, power+SPI routed (DRC 0 errors); small nets handed to ET; JLCPCB-class 0.2 mm rules
- removed SW1 (bench button), J21 (2nd cell -> harness), D1 (VBUS ESD on U12's spare channel)
- router: rip-up/reroute + negotiated congestion options (neither finished the small nets at 0.3 mm)
- design notes: hand-off list for ET, fab rules, layout-driven changes; BoM ~EUR 102/device

Co-Authored-By: Claude Opus 5.5 <noreply@anthropic.com>
Claude-Session: https://claude.ai/code/session_01Dy4TuRNF8V28KreA3jwCtM
Parts:
- removed SW1: bench GO/STOP, Button_Switch_THT:SW_PUSH_6mm, symbol Switch:SW_Push
Other:
- note added: "J10: panel button E-Switch PS1024ABLK (momentary). Bench: plug the panel button into J10 (or bridge its two pins); no on-board button. J11: role toggle E-Switch 100SP1T1B1M1QEH, closed = TX; may stay unfitted until Atenea Q8 (open = RX). J12: mode toggle E-Switch 100SP3T1B1M1QEH ON-OFF-ON: 1 NM, 2 common (GND), 3 MRM; centre = SRI."
- note removed: "J10: panel button E-Switch PS1024ABLK (momentary). SW1: bench button in parallel with J10. J11: role toggle E-Switch 100SP1T1B1M1QEH, closed = TX; may stay unfitted until Atenea Q8 (open = RX). J12: mode toggle E-Switch 100SP3T1B1M1QEH ON-OFF-ON: 1 NM, 2 common (GND), 3 MRM; centre = SRI."
