File: hw/sp4-breakout/sp4-breakout.kicad_pcb (KiCad board)
At the start: 2 copper layers, 31 x 37.5 mm, 8 parts, among them J1 nRF24 header, J2 3V3 bench supply, U1 E01-ML01SP4

Commit message: SP4 breakout: 2.0 mm header pads and no pour between C1's pads (UPC lab rules)
- J1/J2 use teamc:PinHeader_1x08/1x02_P2.54mm_Vertical_Pad2.0mm, written by
  build_breakout.py from the stock headers (1.7 -> 2.0 mm pads, 1.0 mm drill
  kept, pin 1 square): hole + 1.0 mm, 0.54 mm between pads at 2.54 mm pitch.
  A library copy rather than a board override, so DRC's library-parity check
  stays clean.
- FR10: a no-fill rule area in C1's 2.1 mm pad gap (the only SMD gap the pour
  reached); SP4 castellations and the 0805 gaps had no pour.
- build_breakout.py restores the lab floor (0.3 mm clearance/track, 2 thermal
  spokes) after set_project_rules, which lowered it for the carrier.
- Regenerated board, schematic, fab/ and the gerber zip: ERC 0, DRC 0
  violations / 0 unconnected / 0 parity (all severities). Footprint
  positions and the 30 tracks (0.5/0.6 mm) unchanged.

Co-Authored-By: Claude Opus 5.5 <noreply@anthropic.com>
Claude-Session: https://claude.ai/code/session_01PKzvcoWGaf5niy6TrXYsya
Parts:
- J1: footprint Connector_PinHeader_2.54mm:PinHeader_1x08_P2.54mm_Vertical -> teamc:PinHeader_1x08_P2.54mm_Vertical_Pad2.0mm
- J2: footprint Connector_PinHeader_2.54mm:PinHeader_1x02_P2.54mm_Vertical -> teamc:PinHeader_1x02_P2.54mm_Vertical_Pad2.0mm
Changed lines of the file:
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@@
 				(font
 					(size 1.27 1.27)
+					(thickness 0.15)
 				)
 			)
@@
 				(font
 					(size 1.27 1.27)
+					(thickness 0.15)
 				)
 			)
@@
 		)
 	)
-	(footprint "Connector_PinHeader_2.54mm:PinHeader_1x02_P2.54mm_Vertical"
+	(footprint "teamc:PinHeader_1x02_P2.54mm_Vertical_Pad2.0mm"
 		(layer "B.Cu")
 		(at 111.5 100 -90)
-		(descr "Through hole straight pin header, 1x02, 2.54mm pitch, single row")
-		(tags "Through hole pin header THT 1x02 2.54mm single row")
+		(descr "1x02 2.54 mm pin header, vertical, 2.0 mm pads on the 1.0 mm drill (from the KiCad PinHeader_1x02_P2.54mm_Vertical; larger pads for the UPC lab's unplated, hand-soldered holes)")
+		(tags "pin header 2.54 mm Team C lab")
 		(property "Reference" "J2"
 			(at 0 2.38 90)
@@
 		)
 		(property "MPN" "1x02 2.54 mm pin header"
-			(at 0 0 90)
+			(at 0 0 0)
 			(layer "B.SilkS")
 			(hide yes)
@@
 					(thickness 0.15)
 				)
-				(justify mirror)
 			)
 		)
@@
 		(pad "1" thru_hole rect
 			(at 0 0 270)
-			(size 1.7 1.7)
+			(size 2 2)
 			(drill 1)
 			(layers "*.Cu" "*.Mask")
@@
 		(pad "2" thru_hole circle
 			(at 0 -2.54 270)
-			(size 1.7 1.7)
+			(size 2 2)
 			(drill 1)
 			(layers "*.Cu" "*.Mask")
@@
 		)
 	)
-	(footprint "Connector_PinHeader_2.54mm:PinHeader_1x08_P2.54mm_Vertical"
+	(footprint "teamc:PinHeader_1x08_P2.54mm_Vertical_Pad2.0mm"
 		(layer "B.Cu")
 		(at 110.795 79 90)
-		(descr "Through hole straight pin header, 1x08, 2.54mm pitch, single row")
-		(tags "Through hole pin header THT 1x08 2.54mm single row")
+		(descr "1x08 2.54 mm pin header, vertical, 2.0 mm pads on the 1.0 mm drill (from the KiCad PinHeader_1x08_P2.54mm_Vertical; larger pads for the UPC lab's unplated, hand-soldered holes)")
+		(tags "pin header 2.54 mm Team C lab")
 		(property "Reference" "J1"
 			(at 0 2.38 270)
@@
 		)
 		(property "MPN" "1x08 2.54 mm pin header"
-			(at 0 0 270)
+			(at 0 0 0)
 			(layer "B.SilkS")
 			(hide yes)
@@
 					(thickness 0.15)
 				)
-				(justify mirror)
 			)
 		)
@@
 		(pad "1" thru_hole rect
 			(at 0 0 90)
-			(size 1.7 1.7)
+			(size 2 2)
 			(drill 1)
 			(layers "*.Cu" "*.Mask")
@@
 		(pad "2" thru_hole circle
 			(at 0 -2.54 90)
-			(size 1.7 1.7)
+			(size 2 2)
 			(drill 1)
 			(layers "*.Cu" "*.Mask")
@@
 		(pad "3" thru_hole circle
 			(at 0 -5.08 90)
-			(size 1.7 1.7)
+			(size 2 2)
 			(drill 1)
 			(layers "*.Cu" "*.Mask")
@@
 		(pad "4" thru_hole circle
 			(at 0 -7.62 90)
-			(size 1.7 1.7)
+			(size 2 2)
 			(drill 1)
 			(layers "*.Cu" "*.Mask")
@@
 		(pad "5" thru_hole circle
 			(at 0 -10.16 90)
-			(size 1.7 1.7)
+			(size 2 2)
 			(drill 1)
 			(layers "*.Cu" "*.Mask")
@@
 		(pad "6" thru_hole circle
 			(at 0 -12.7 90)
-			(size 1.7 1.7)
+			(size 2 2)
 			(drill 1)
 			(layers "*.Cu" "*.Mask")
@@
 		(pad "7" thru_hole circle
 			(at 0 -15.24 90)
-			(size 1.7 1.7)
+			(size 2 2)
 			(drill 1)
 			(layers "*.Cu" "*.Mask")
@@
 		(pad "8" thru_hole circle
 			(at 0 -17.78 90)
-			(size 1.7 1.7)
+			(size 2 2)
 			(drill 1)
 			(layers "*.Cu" "*.Mask")
@@
 	)
 	(segment
+		(start 104.445 88.9)
+		(end 108.255 88.9)
+		(width 0.5)
+		(layer "F.Cu")
+		(net "/VCC")
+	)
+	(segment
+		(start 108.255 88.9)
+		(end 112.399999 88.9)
+		(width 0.6)
+		(layer "F.Cu")
+		(net "/VCC")
+	)
+	(segment
+		(start 112.399999 88.9)
+		(end 114.6 88.9)
+		(width 0.6)
+		(layer "F.Cu")
+		(net "/VCC")
+	)
+	(segment
 		(start 111.5 96)
 		(end 112.399999 96)
@@
 	)
 	(segment
-		(start 104.445 88.9)
-		(end 108.255 88.9)
-		(width 0.5)
+		(start 108.255 79)
+		(end 108.255 84.6)
+		(width 0.6)
+		(layer "F.Cu")
+		(net "/VCC")
+	)
+	(segment
+		(start 111.5 100)
+		(end 111.5 96)
+		(width 0.6)
 		(layer "F.Cu")
 		(net "/VCC")
@@
 	)
 	(segment
-		(start 112.399999 88.9)
-		(end 114.6 88.9)
-		(width 0.6)
-		(layer "F.Cu")
-		(net "/VCC")
-	)
-	(segment
-		(start 108.255 88.9)
-		(end 112.399999 88.9)
-		(width 0.6)
-		(layer "F.Cu")
-		(net "/VCC")
-	)
-	(segment
-		(start 111.5 100)
-		(end 111.5 96)
+		(start 110.5625 84.6)
+		(end 108.255 84.6)
 		(width 0.6)
 		(layer "F.Cu")
@@
 	)
 	(segment
+		(start 108.255 84.6)
+		(end 108.255 87.2)
+		(width 0.6)
+		(layer "F.Cu")
+		(net "/VCC")
+	)
+	(segment
+		(start 112.399999 96)
+		(end 112.399999 88.9)
+		(width 0.6)
+		(layer "F.Cu")
+		(net "/VCC")
+	)
+	(segment
 		(start 108.255 87.2)
 		(end 108.255 88.9)
@@
 	)
 	(segment
-		(start 108.255 79)
-		(end 108.255 84.6)
-		(width 0.6)
-		(layer "F.Cu")
-		(net "/VCC")
-	)
-	(segment
-		(start 108.255 84.6)
-		(end 108.255 87.2)
-		(width 0.6)
-		(layer "F.Cu")
-		(net "/VCC")
-	)
-	(segment
-		(start 110.5625 84.6)
-		(end 108.255 84.6)
-		(width 0.6)
-		(layer "F.Cu")
-		(net "/VCC")
-	)
-	(segment
-		(start 112.399999 96)
-		(end 112.399999 88.9)
-		(width 0.6)
-		(layer "F.Cu")
-		(net "/VCC")
+		(start 103.175 90.9)
+		(end 103.175 88.5)
+		(width 0.5)
+		(layer "F.Cu")
+		(net "/CE")
+	)
+	(segment
+		(start 105.715 85.96)
+		(end 105.715 79)
+		(width 0.5)
+		(layer "F.Cu")
+		(net "/CE")
 	)
 	(segment
@@
 	)
 	(segment
-		(start 103.175 90.9)
-		(end 103.175 88.5)
+		(start 101.905 88.5)
+		(end 103.175 87.23)
 		(width 0.5)
 		(layer "F.Cu")
-		(net "/CE")
-	)
-	(segment
-		(start 105.715 85.96)
-		(end 105.715 79)
-		(width 0.5)
-		(layer "F.Cu")
-		(net "/CE")
+		(net "/CSN")
 	)
 	(segment
@@
 	)
 	(segment
-		(start 101.905 88.5)
-		(end 103.175 87.23)
+		(start 100.635 88.5)
+		(end 100.635 79)
 		(width 0.5)
 		(layer "F.Cu")
-		(net "/CSN")
+		(net "/SCK")
 	)
 	(segment
@@
 	)
 	(segment
-		(start 100.635 88.5)
-		(end 100.635 79)
+		(start 98.095 87.23)
+		(end 98.095 79)
 		(width 0.5)
 		(layer "F.Cu")
-		(net "/SCK")
+		(net "/MOSI")
+	)
+	(segment
+		(start 99.365 88.5)
+		(end 98.095 87.23)
+		(width 0.5)
+		(layer "F.Cu")
+		(net "/MOSI")
 	)
 	(segment
@@
 	)
 	(segment
-		(start 98.095 87.23)
-		(end 98.095 79)
+		(start 98.095 90.9)
+		(end 98.095 88.5)
 		(width 0.5)
 		(layer "F.Cu")
-		(net "/MOSI")
-	)
-	(segment
-		(start 99.365 88.5)
-		(end 98.095 87.23)
-		(width 0.5)
-		(layer "F.Cu")
-		(net "/MOSI")
+		(net "/MISO")
 	)
 	(segment
@@
 	)
 	(segment
-		(start 98.095 90.9)
-		(end 98.095 88.5)
+		(start 93.015 84.69)
+		(end 93.015 79)
 		(width 0.5)
 		(layer "F.Cu")
-		(net "/MISO")
+		(net "/IRQ")
 	)
 	(segment
@@
 		(net "/IRQ")
 	)
-	(segment
-		(start 93.015 84.69)
-		(end 93.015 79)
-		(width 0.5)
-		(layer "F.Cu")
-		(net "/IRQ")
-	)
 	(zone
+		(layer "F.Cu")
+		(name "C1_no_pour")
+		(hatch edge 0.5)
+		(connect_pads
+			(clearance 0)
+		)
+		(min_thickness 0.25)
+		(keepout
+			(tracks allowed)
+			(vias allowed)
+			(pads allowed)
+			(copperpour not_allowed)
+			(footprints allowed)
+		)
+		(placement
+			(enabled no)
+			(sheetname "")
+		)
+		(fill
+			(thermal_gap 0.5)
+			(thermal_bridge_width 0.5)
+			(island_removal_mode 0)
+		)
+		(polygon
+			(pts
+				(xy 113.8 92.55) (xy 115.4 92.55) (xy 115.4 94.65) (xy 113.8 94.65)
+			)
+		)
+	)
+	(zone
