File: hw/teamc-carrier-lab/power.kicad_sch (KiCad schematic)
At the start: 24 parts, among them J20 BATT 18650, J22 PWR toggle, J23 TP4056 B+/B-, Q1 DMP2035U, Q2 2N7002, U2 Pololu U3V70F5 5V boost, U3 Pololu ideal diode 20A, U4 AP2112K-3.3, U6 Adafruit MAX17048 fuel gauge

Commit message: Carrier rev B (UPC lab): placed and routed on one copper layer, DRC 0/0/0
- place_carrier_lab.py: fixed floorplan (power right, J1 centre, SP4 socket top-left
  edge, UI leads left edge, fuel gauge bottom-left); provisional 100 x 80 mm outline
  until the box is measured.
- linkroute.py: single-layer grid router whose second "layer" is straight wire links
  (bare wire on the component side between two unplated holes).
- route_carrier_lab.py: hand-coded power path, SCK swap under R84/R83, left half; the
  rest routed in a topology order, --search over the band-net orders.
- finish_carrier_lab.py: GND pour (0.4 mm), FR10 no-fill areas, M3 keep-outs, ground
  island joins, links -> W parts (one-pin symbol, WireLink footprint with jumper pads).
- fab_carrier_lab.py: F.Cu + Edge.Cuts gerbers, drill, 1:1 copper PDFs, assembly and
  schematic PDFs, zip; renders; build_bom.py --rev b -> hw/BOM_revB.csv (~EUR 139).
- Schematic changes for one layer (documented on the sheets and in DESIGN_NOTES):
  1206 R/C, no UI pull-ups, 4 x SMF5.0A instead of SP0504, R80 to 3V3_RADIO, no R81,
  no C71/TP10/TP2 (C12 10 uF), 3V3_PI from J1 pin 1, FG_ALRT not routed, LED return
  on pin 25, J1 GND pins 20/30/34/39 unused, J23 on BAT_IN.
- ERC 0; DRC 0 violations / 0 unconnected / 0 parity (silk/mask checks off: the lab
  board has neither); 10 wire links (138 mm).

Co-Authored-By: Claude Opus 5.5 <noreply@anthropic.com>
Claude-Session: https://claude.ai/code/session_01M3xdFsssmBw3o2iBWKaKwo
Parts:
- removed TP2: 5V_PI, TestPoint:TestPoint_Loop_D2.50mm_Drill1.0mm, symbol Connector:TestPoint
- C10, C18: footprint Capacitor_SMD:C_0805_2012Metric_Pad1.18x1.45mm_HandSolder -> Capacitor_SMD:C_1206_3216Metric_Pad1.33x1.80mm_HandSolder; MPN CL21B104KBCNNNC -> CL31B104KBCNNNC
- C11: footprint Capacitor_SMD:C_0805_2012Metric_Pad1.18x1.45mm_HandSolder -> Capacitor_SMD:C_1206_3216Metric_Pad1.33x1.80mm_HandSolder; MPN CL21A106KAYNNNE -> CL31A106KAHNNNE
- C12: value 1u X7R -> 10u X5R; footprint Capacitor_SMD:C_0805_2012Metric_Pad1.18x1.45mm_HandSolder -> Capacitor_SMD:C_1206_3216Metric_Pad1.33x1.80mm_HandSolder; MPN CL21B105KBFNNNE -> CL31A106KAHNNNE
- R1: footprint Resistor_SMD:R_0805_2012Metric_Pad1.20x1.40mm_HandSolder -> Resistor_SMD:R_1206_3216Metric_Pad1.30x1.75mm_HandSolder; MPN RC0805FR-0710KL -> RC1206FR-0710KL
- R8: footprint Resistor_SMD:R_0805_2012Metric_Pad1.20x1.40mm_HandSolder -> Resistor_SMD:R_1206_3216Metric_Pad1.30x1.75mm_HandSolder; MPN RC0805FR-07100KL -> RC1206FR-07100KL
- R9: footprint Resistor_SMD:R_0805_2012Metric_Pad1.20x1.40mm_HandSolder -> Resistor_SMD:R_1206_3216Metric_Pad1.30x1.75mm_HandSolder; MPN RC0805FR-071KL -> RC1206FR-071KL
Connections:
- net BAT_IN: now also J23.1 (Pin_1)
- net GND: no longer U6.2 (Pin_2)
- net VBAT: no longer J23.1 (Pin_1)
- net FG_ALRT: no longer names the net of U6.5 (Pin_5)
- no-connect marks 1 -> 3
Other:
- note added: "Protected 18650 (PCM inside, trip >= 3 A) in a holder on the box floor, JST-VH lead to J20. Q1: body diode conducts for a correct cell, then VGS = -VBAT turns it on; a reversed cell is blocked. DMP2035U <= 45 mΩ at -2.5 V (AO3401A ~85 mΩ: ~0.25 V at 3 A). C5: bulk at the boost input (Pololu asks for >= 33 uF when the cell is on a lead). Charger (J23): rev B on BAT_IN, beside J20 (the cell lead)."
- note added: "Rev B: no 5V_PI loop (rev A TP2): probe D2's cathode pad."
- note added: "The chip runs from the cell (SJ2 bridged VDD-Bat as shipped); header VIN only feeds its 10 k pull-ups on SCL/SDA/INT and the LED (cut SJ1 to save ~0.1 mA): VIN = 3V3_PI (rev B: from J1 pin 1). Cell sense through the JP2 Bat/GND pair (2-pin header, Kelvin track from Q1's source), not a JST-PH lead. QSTART unused (10 k to GND on the module). INT (alert) not routed in rev B: the software polls SOC o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"
- note added: "~0.1 V dropout at 150 mA (600 mA part). EN from 3V3_PI: the radio is off whenever the Pi is off (else the SP4 in RX drains ~26 mA from the cell with the box 'off'). The breakout adds 110 uF at the module. C12 10 uF (rev A 1 uF + 10 uF C71 at the socket): the socket is 6 mm away on the lab board; AP2112 needs >= 1 uF."
- note removed: "Protected 18650 (PCM inside, trip >= 3 A) in a holder on the box floor, JST-VH lead to J20. Q1: body diode conducts for a correct cell, then VGS = -VBAT turns it on; a reversed cell is blocked. DMP2035U <= 45 mΩ at -2.5 V (AO3401A ~85 mΩ: ~0.25 V at 3 A). C5: bulk at the boost input (Pololu asks for >= 33 uF when the cell is on a lead). Charger (J23) on VBAT: Q1 conducts both ways once on."
- note removed: "The chip runs from the cell (SJ2 bridged VDD-Bat as shipped); header VIN only feeds its 10 k pull-ups on SCL/SDA/INT and the LED (cut SJ1 to save ~0.1 mA): VIN = 3V3_PI. Cell sense through the JP2 Bat/GND pair (2-pin header, Kelvin track from Q1's source), not a JST-PH lead. QSTART unused (10 k to GND on the module). No level shifting needed at 3.3 V. Software: never set MODE.EnSleep."
- note removed: "~0.1 V dropout at 150 mA (600 mA part). EN from 3V3_PI: the radio is off whenever the Pi is off (else the SP4 in RX drains ~26 mA from the cell with the box 'off'). The breakout adds 110 uF at the module."

Commit message: Carrier rev B review fixes: charger on VBAT, insulated links, SPI at 4 MHz
- J23 (TP4056 lead) back on VBAT behind F1/Q1: placed between the VBAT line and
  C5, GND to C5's ground pad, R1 now returns to J20's GND pin. A reversed cell no
  longer reaches the charger and the lead is fused.
- Wire links: insulated 22 AWG solid hook-up wire, not bare (schematic note, W
  MPN, WireLink footprint text, BoM, shopping list).
- Ribbon grounds: tying J1 20/25 to the pour was tried; the inner pocket of J1's
  escape ring (LEDs, pins 20/25) has no legal wire link, the outer pockets would
  cost 3 more. Kept as before and SPI defaults to 4 MHz instead (teamc-node
  --spi-hz, NRF24_LINUX_CFG_DEFAULT; was 8 MHz) until T2 is clean; flying-wire
  fallback documented.
- Pipeline rerun twice: ERC 0, DRC 0/0/0, one copper layer, no vias, 10 links;
  fab zip, 1:1 PDFs, renders and BOM_revB.csv (EUR 139.01) regenerated.
- fw 318, proto all scenarios + 116 usb, linux builds, phy_config OK.

Co-Authored-By: Claude Opus 5.5 <noreply@anthropic.com>
Claude-Session: https://claude.ai/code/session_01PKzvcoWGaf5niy6TrXYsya
Connections:
- net BAT_IN: no longer J23.1 (Pin_1)
- net VBAT: now also J23.1 (Pin_1)
Other:
- note added: "Protected 18650 (PCM inside, trip >= 3 A) in a holder on the box floor, JST-VH lead to J20. Q1: body diode conducts for a correct cell, then VGS = -VBAT turns it on; a reversed cell is blocked. DMP2035U <= 45 mΩ at -2.5 V (AO3401A ~85 mΩ: ~0.25 V at 3 A). C5: bulk at the boost input (Pololu asks for >= 33 uF when the cell is on a lead). Charger (J23) on VBAT, behind F1 and Q1 (review 23-Oct): a r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"
- note removed: "Protected 18650 (PCM inside, trip >= 3 A) in a holder on the box floor, JST-VH lead to J20. Q1: body diode conducts for a correct cell, then VGS = -VBAT turns it on; a reversed cell is blocked. DMP2035U <= 45 mΩ at -2.5 V (AO3401A ~85 mΩ: ~0.25 V at 3 A). C5: bulk at the boost input (Pololu asks for >= 33 uF when the cell is on a lead). Charger (J23): rev B on BAT_IN, beside J20 (the cell lead)."
Changed lines of the file:
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@@
 		)
 	)
-	(label "BAT_IN"
+	(global_label "VBAT"
+		(shape passive)
 		(at 152.4 38.1 180)
 		(fields_autoplaced yes)
@@
 				(size 1.27 1.27)
 			)
-			(justify right bottom)
+			(justify right)
 		)
 	)
@@
 		)
 	)
-	(text "Protected 18650 (PCM inside, trip >= 3 A) in a holder on the box floor, JST-VH lead to J20.\nQ1: body diode conducts for a correct cell, then VGS = -VBAT turns it on; a reversed cell is blocked.\nDMP2035U <= 45 mΩ at -2.5 V (AO3401A ~85 mΩ: ~0.25 V at 3 A). C5: bulk at the boost input (Pololu asks\nfor >= 33 uF when the cell is on a lead). Charger (J23): rev B on BAT_IN, beside J20 (the cell lead)."
+	(text "Protected 18650 (PCM inside, trip >= 3 A) in a holder on the box floor, JST-VH lead to J20.\nQ1: body diode conducts for a correct cell, then VGS = -VBAT turns it on; a reversed cell is blocked.\nDMP2035U <= 45 mΩ at -2.5 V (AO3401A ~85 mΩ: ~0.25 V at 3 A). C5: bulk at the boost input (Pololu asks\nfor >= 33 uF when the cell is on a lead). Charger (J23) on VBAT, behind F1 and Q1 (review 23-Oct): a\nreversed cell never reaches the TP4056, and a short in the charger lead is fused. Q1 conducts both ways once on."
 		(exclude_from_sim no)
 		(at 15.24 91.44 0)
