File: hw/teamc-carrier-lab/teamc-carrier-lab.kicad_pcb (KiCad board)
At the start: 2 copper layers, 100 x 80 mm, 59 parts, among them J1 RPi GPIO ribbon, J10 GO/STOP button, J11 role toggle, J12 mode toggle, J13 UART console, J20 BATT 18650, J22 PWR toggle, J23 TP4056 B+/B-, J30 SP4 breakout, Q1 DMP2035U, Q2 2N7002, U11 SP0504BAHTG, U2 Pololu U3V70F5 5V boost, U3 Pololu ideal diode 20A, U4 AP2112K-3.3, U6 Adafruit MAX17048 fuel gauge

Commit message: Carrier rev B (UPC lab): placed and routed on one copper layer, DRC 0/0/0
- place_carrier_lab.py: fixed floorplan (power right, J1 centre, SP4 socket top-left
  edge, UI leads left edge, fuel gauge bottom-left); provisional 100 x 80 mm outline
  until the box is measured.
- linkroute.py: single-layer grid router whose second "layer" is straight wire links
  (bare wire on the component side between two unplated holes).
- route_carrier_lab.py: hand-coded power path, SCK swap under R84/R83, left half; the
  rest routed in a topology order, --search over the band-net orders.
- finish_carrier_lab.py: GND pour (0.4 mm), FR10 no-fill areas, M3 keep-outs, ground
  island joins, links -> W parts (one-pin symbol, WireLink footprint with jumper pads).
- fab_carrier_lab.py: F.Cu + Edge.Cuts gerbers, drill, 1:1 copper PDFs, assembly and
  schematic PDFs, zip; renders; build_bom.py --rev b -> hw/BOM_revB.csv (~EUR 139).
- Schematic changes for one layer (documented on the sheets and in DESIGN_NOTES):
  1206 R/C, no UI pull-ups, 4 x SMF5.0A instead of SP0504, R80 to 3V3_RADIO, no R81,
  no C71/TP10/TP2 (C12 10 uF), 3V3_PI from J1 pin 1, FG_ALRT not routed, LED return
  on pin 25, J1 GND pins 20/30/34/39 unused, J23 on BAT_IN.
- ERC 0; DRC 0 violations / 0 unconnected / 0 parity (silk/mask checks off: the lab
  board has neither); 10 wire links (138 mm).

Co-Authored-By: Claude Opus 5.5 <noreply@anthropic.com>
Claude-Session: https://claude.ai/code/session_01M3xdFsssmBw3o2iBWKaKwo
Parts:
- removed C71: 10u X5R, Capacitor_SMD:C_0805_2012Metric_Pad1.18x1.45mm_HandSolder
- removed R50, R51, R52, R53, R81: 10k, Resistor_SMD:R_0805_2012Metric_Pad1.20x1.40mm_HandSolder
- removed TP10: 3V3_RADIO, TestPoint:TestPoint_Loop_D2.50mm_Drill1.0mm
- removed TP2: 5V_PI, TestPoint:TestPoint_Loop_D2.50mm_Drill1.0mm
- removed U11: SP0504BAHTG, Package_TO_SOT_SMD:SOT-23-5
- added D12: SMF5.0A, Diode_SMD:D_SMF, F.Cu at (58.5, 115.0)
- added D13: SMF5.0A, Diode_SMD:D_SMF, F.Cu at (58.5, 106.5)
- added D14: SMF5.0A, Diode_SMD:D_SMF, F.Cu at (58.5, 93.5)
- added D15: SMF5.0A, Diode_SMD:D_SMF, F.Cu at (61.5, 95.5)
- added W1: wire link 34.5 mm, teamc:WireLink_L34.5mm, B.Cu at (66.0, 85.5)
- added W10: wire link 5.0 mm, teamc:WireLink_L5.0mm, B.Cu at (107.0, 62.0)
- added W2: wire link 8.0 mm, teamc:WireLink_L8.0mm, B.Cu at (54.0, 61.0)
- added W3: wire link 8.5 mm, teamc:WireLink_L8.5mm, B.Cu at (61.0, 111.5)
- added W4: wire link 13.0 mm, teamc:WireLink_L13.0mm, B.Cu at (70.0, 61.0)
- added W5: wire link 19.5 mm, teamc:WireLink_L19.5mm, B.Cu at (76.0, 54.0)
- added W6: wire link 5.0 mm, teamc:WireLink_L5.0mm, B.Cu at (104.0, 62.5)
- added W7: wire link 18.5 mm, teamc:WireLink_L18.5mm, B.Cu at (79.0, 81.5)
- added W8: wire link 15.0 mm, teamc:WireLink_L15.0mm, B.Cu at (64.0, 78.5)
- added W9: wire link 10.5 mm, teamc:WireLink_L10.5mm, B.Cu at (88.5, 58.5)
- C10, C11, C18, C50, C51, C52, C53: footprint Capacitor_SMD:C_0805_2012Metric_Pad1.18x1.45mm_HandSolder -> Capacitor_SMD:C_1206_3216Metric_Pad1.33x1.80mm_HandSolder
- C12: value 1u X7R -> 10u X5R; footprint Capacitor_SMD:C_0805_2012Metric_Pad1.18x1.45mm_HandSolder -> Capacitor_SMD:C_1206_3216Metric_Pad1.33x1.80mm_HandSolder
- H30, J1, J10, J11, J12, J13, J20, J22, J23, J30, MH1, MH2, MH3, MH4, TP1, TP3, U2, U3, U6: moved to B.Cu
- R1, R54, R55, R56, R57, R60, R61, R8, R80, R82, R83, R84, R9: footprint Resistor_SMD:R_0805_2012Metric_Pad1.20x1.40mm_HandSolder -> Resistor_SMD:R_1206_3216Metric_Pad1.30x1.75mm_HandSolder
- moved U4 452.9 mm to (61.0, 64.0)
- moved U6 406.1 mm to (78.4, 116.2), turned to -90 degrees
- moved U2 403.4 mm to (128.7, 87.8), turned to -90 degrees
- moved TP1 389.3 mm to (144.0, 61.0)
- moved U3 379.0 mm to (118.1, 121.3), turned to 180 degrees
- moved R9 375.8 mm to (113.5, 69.0)
- moved R80 360.9 mm to (67.0, 53.2)
- moved TP3 360.5 mm to (140.0, 114.0)
- moved R84 346.5 mm to (90.0, 94.6), turned to 180 degrees
- moved R83 336.2 mm to (90.0, 97.1), turned to 180 degrees
- moved R8 329.3 mm to (118.0, 67.3), turned to -90 degrees
- moved R82 328.1 mm to (84.0, 98.7), turned to 180 degrees
- moved R61 314.9 mm to (90.0, 78.9)
- moved R60 301.8 mm to (90.0, 84.4)
- moved R57 288.2 mm to (67.5, 97.0)
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Connections:
- D10 pad 1: GND -> LED_RTN
- D11 pad 1: GND -> LED_RTN
- J1 pad 1: unconnected-(J1-Pin_1-Pad1) -> 3V3_PI
- J1 pad 17: 3V3_PI -> unconnected-(J1-Pin_17-Pad17)
- J1 pad 20: GND -> unconnected-(J1-Pin_20-Pad20)
- J1 pad 22: FG_ALRT -> unconnected-(J1-Pin_22-Pad22)
- J1 pad 25: GND -> LED_RTN
- J1 pad 30: GND -> unconnected-(J1-Pin_30-Pad30)
- J1 pad 34: GND -> unconnected-(J1-Pin_34-Pad34)
- J1 pad 39: GND -> unconnected-(J1-Pin_39-Pad39)
- J23 pad 1: VBAT -> /power/BAT_IN
- R80 pad 1: 3V3_PI -> 3V3_RADIO
- U6 pad 2: GND -> unconnected-(U6-Pin_2-Pad2)
- U6 pad 5: FG_ALRT -> unconnected-(U6-Pin_5-Pad5)
Routing:
- net VBAT: track 0.00 -> 237.6 mm
- net GND: track 0.00 -> 208.9 mm
- net SW_MODE_NM: track 0.00 -> 95.9 mm
- net 3V3_PI: track 0.00 -> 73.5 mm
- net RADIO_CE: track 0.00 -> 61.8 mm
- net RADIO_CSN: track 0.00 -> 51.0 mm
- net RADIO_IRQ: track 0.00 -> 49.6 mm
- net /radio/SCK_R: track 0.00 -> 43.3 mm
- net /radio/MOSI_R: track 0.00 -> 43.2 mm
- net SW_MODE_MRM: track 0.00 -> 42.1 mm
- net 5V_PI: track 0.00 -> 40.5 mm
- net /radio/MISO_R: track 0.00 -> 39.5 mm
- net BTN_TXRX: track 0.00 -> 27.4 mm
- net 5V_BOOST: track 0.00 -> 27.3 mm
- net SW_ROLE: track 0.00 -> 25.0 mm
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- added copper zone on F.Cu, net GND
Other:
- board text added: "SP4 breakout above (IPEX end)"

Commit message: Carrier rev B review fixes: charger on VBAT, insulated links, SPI at 4 MHz
- J23 (TP4056 lead) back on VBAT behind F1/Q1: placed between the VBAT line and
  C5, GND to C5's ground pad, R1 now returns to J20's GND pin. A reversed cell no
  longer reaches the charger and the lead is fused.
- Wire links: insulated 22 AWG solid hook-up wire, not bare (schematic note, W
  MPN, WireLink footprint text, BoM, shopping list).
- Ribbon grounds: tying J1 20/25 to the pour was tried; the inner pocket of J1's
  escape ring (LEDs, pins 20/25) has no legal wire link, the outer pockets would
  cost 3 more. Kept as before and SPI defaults to 4 MHz instead (teamc-node
  --spi-hz, NRF24_LINUX_CFG_DEFAULT; was 8 MHz) until T2 is clean; flying-wire
  fallback documented.
- Pipeline rerun twice: ERC 0, DRC 0/0/0, one copper layer, no vias, 10 links;
  fab zip, 1:1 PDFs, renders and BOM_revB.csv (EUR 139.01) regenerated.
- fw 318, proto all scenarios + 116 usb, linux builds, phy_config OK.

Co-Authored-By: Claude Opus 5.5 <noreply@anthropic.com>
Claude-Session: https://claude.ai/code/session_01PKzvcoWGaf5niy6TrXYsya
Parts:
- moved J23 36.0 mm to (145.5, 70.0)
Connections:
- J23 pad 1: /power/BAT_IN -> VBAT
Routing:
- net /power/BAT_IN: track 13.1 -> 3.51 mm
- net GND: track 208.9 -> 202.1 mm
- net VBAT: track 237.6 -> 242.1 mm
