File: hw/teamc-carrier-simple/pi_link.kicad_sch (KiCad schematic)
At the start: 6 parts, among them J1 RPi GPIO ribbon, J13 UART console

Commit message: Carrier rev C (simple): checkpoint 3 - placed and routed on one copper layer, DRC 0/0/0, 4 wire links
120 x 66 mm (box not measured yet: hw/scripts/layout_carrier_simple.py rebuilds everything after the
outline in place_carrier_simple.py changes). Backbone hand-routed (route_carrier_simple.py), router for
the short branches, GND pour; DRC with schematic parity 0 violations / 0 unconnected / 0 parity, all
severities; ERC 0/0. Tracks 0.8-2.0 mm. Wire links: IRQ over CSN and three ground pockets. Crossings by
tracks between resistor legs (SCK under R84/R83, LED_ACT_A under R61, CSN/IRQ under R57).
Layout-driven schematic changes: input 100 nF caps dropped, C18 at the toggle lead, 7.62 mm resistor
pitch, D1 on 12.7 mm, three M3 holes. Cable-tie slot + edge notch at the cell. 3D models for the
modules, wire links, holder, fuse clips and test points (gen_3d_revc.py; fetch_3d substitutes).
Fab: F.Cu + Edge.Cuts gerbers, drill, 1:1 copper PDFs, assembly PDFs, wire_links.csv, zip; renders.

Co-Authored-By: Claude Opus 5.5 <noreply@anthropic.com>
Parts:
- removed MH4: M3, MountingHole:MountingHole_3.2mm_M3, symbol Mechanical:MountingHole
- added W1: wire link 4.0 mm, teamc:RevC_WireLink_L4.0mm, symbol Connector_Generic:Conn_01x01
- added W2: wire link 7.2 mm, teamc:RevC_WireLink_L7.2mm, symbol Connector_Generic:Conn_01x01
- added W3: wire link 6.0 mm, teamc:RevC_WireLink_L6.0mm, symbol Connector_Generic:Conn_01x01
- added W4: wire link 5.7 mm, teamc:RevC_WireLink_L5.7mm, symbol Connector_Generic:Conn_01x01
Connections:
- net GND: now also W1.1 (Pin_1), W2.1 (Pin_1), W3.1 (Pin_1)
- net RADIO_IRQ: now also W4.1 (Pin_1)
Other:
- note added: "WIRE LINKS (one copper layer): INSULATED 22 AWG solid tinned copper wire on the component side between two unplated 1.0 mm holes, ends stripped ~3 mm, soldered on the copper side; lay it flat, glue it for the drop test. Positions and lengths: hw/teamc-carrier-simple/links.json and the assembly drawing."
