File: hw/teamc-carrier-simple/teamc-carrier-simple.kicad_pcb (KiCad board)
At the start: 2 copper layers, 120 x 63 mm, 46 parts, among them J1 RPi GPIO ribbon, J10 GO/STOP button, J11 role toggle, J12 mode toggle, J13 UART console, J14 LED lead, J22 PWR toggle, J23 charger BAT+/BAT-, J30 SP4 breakout, U2 Pololu U3V70F5 5V boost, U3 Pololu ideal diode 20A, U4 MCP1700-3302E/TO, U6 Adafruit MAX17048 fuel gauge

Commit message: Carrier rev C (simple): checkpoint 3 - placed and routed on one copper layer, DRC 0/0/0, 4 wire links
120 x 66 mm (box not measured yet: hw/scripts/layout_carrier_simple.py rebuilds everything after the
outline in place_carrier_simple.py changes). Backbone hand-routed (route_carrier_simple.py), router for
the short branches, GND pour; DRC with schematic parity 0 violations / 0 unconnected / 0 parity, all
severities; ERC 0/0. Tracks 0.8-2.0 mm. Wire links: IRQ over CSN and three ground pockets. Crossings by
tracks between resistor legs (SCK under R84/R83, LED_ACT_A under R61, CSN/IRQ under R57).
Layout-driven schematic changes: input 100 nF caps dropped, C18 at the toggle lead, 7.62 mm resistor
pitch, D1 on 12.7 mm, three M3 holes. Cable-tie slot + edge notch at the cell. 3D models for the
modules, wire links, holder, fuse clips and test points (gen_3d_revc.py; fetch_3d substitutes).
Fab: F.Cu + Edge.Cuts gerbers, drill, 1:1 copper PDFs, assembly PDFs, wire_links.csv, zip; renders.

Co-Authored-By: Claude Opus 5.5 <noreply@anthropic.com>
Parts:
- removed C50, C51, C52, C53: 100n X7R, teamc:C_Disc_D5.0mm_W2.5mm_P5.00mm_Pad1.8mm
- removed MH4: M3, MountingHole:MountingHole_3.2mm_M3
- added W1: wire link 4.0 mm, teamc:RevC_WireLink_L4.0mm, B.Cu at (57.6, 60.2)
- added W2: wire link 7.2 mm, teamc:RevC_WireLink_L7.2mm, B.Cu at (106.3, 83.0)
- added W3: wire link 6.0 mm, teamc:RevC_WireLink_L6.0mm, B.Cu at (127.0, 53.4)
- added W4: wire link 5.7 mm, teamc:RevC_WireLink_L5.7mm, B.Cu at (108.3, 60.8)
- BT1, C1, C10, C11, C12, C18, C9, F1, H30, J1, J10, J11, J12, J13, J14, J22, J23, J30, MH1, MH2, MH3, TP1, TP2, TP3, TP4, U4: moved to B.Cu
- D1: footprint Diode_THT:D_DO-201AD_P15.24mm_Horizontal -> Diode_THT:D_DO-201AD_P12.70mm_Horizontal; moved to B.Cu
- R54, R55, R56, R57, R60, R61, R80, R82, R83, R84, R9: footprint teamc:R_Axial_DIN0207_L6.3mm_D2.5mm_P10.16mm_Horizontal_Pad1.8mm -> teamc:R_Axial_DIN0207_L6.3mm_D2.5mm_P7.62mm_Horizontal_Pad1.8mm; moved to B.Cu
- U2: footprint teamc:Pololu_U3V70F5_Headers -> teamc:RevC_Pololu_U3V70F5_Headers; moved to B.Cu
- U3: footprint teamc:Pololu_IdealDiode_5388_Headers -> teamc:RevC_Pololu_IdealDiode_5388_Headers; moved to B.Cu
- U6: footprint teamc:Adafruit_MAX17048_5580_Headers -> teamc:RevC_Adafruit_MAX17048_5580_Headers; moved to B.Cu
- moved U4 358.2 mm to (57.0, 65.5)
- moved U3 340.4 mm to (139.1, 56.0), turned to 180 degrees
- moved U6 330.3 mm to (134.2, 82.8)
- moved TP4 325.2 mm to (63.2, 74.5)
- moved U2 315.6 mm to (161.9, 70.8), turned to 90 degrees
- moved TP2 308.9 mm to (59.0, 77.8)
- moved R84 285.5 mm to (78.5, 71.1), turned to 90 degrees
- moved R80 284.8 mm to (64.5, 53.6)
- moved R83 279.7 mm to (74.0, 71.1), turned to 90 degrees
- moved TP3 264.8 mm to (166.8, 105.5)
- moved R82 260.7 mm to (81.5, 80.6), turned to 90 degrees
- moved R57 253.5 mm to (83.5, 55.6), turned to -90 degrees
- moved R9 245.4 mm to (168.3, 100.8), turned to 90 degrees
- moved R61 244.6 mm to (99.5, 75.0), turned to -90 degrees
- moved TP1 243.8 mm to (160.3, 111.0)
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Connections:
- C18 pad 1: /power/PWR_EN -> /power/PWR_SW_J
Routing:
- net 5V_PI: track 0.00 -> 149.4 mm
- net RADIO_CE: track 0.00 -> 105.6 mm
- net SPI_MOSI: track 0.00 -> 77.1 mm
- net SW_ROLE: track 0.00 -> 73.6 mm
- net VBAT: track 0.00 -> 70.4 mm
- net SPI_MISO: track 0.00 -> 67.6 mm
- net RADIO_CSN: track 0.00 -> 55.0 mm
- net BTN_TXRX: track 0.00 -> 50.8 mm
- net SPI_SCK: track 0.00 -> 50.2 mm
- net RADIO_IRQ: track 0.00 -> 41.6 mm
- net 3V3_PI: track 0.00 -> 28.3 mm
- net /radio/SCK_R: track 0.00 -> 25.3 mm
- net 3V3_RADIO: track 0.00 -> 23.0 mm
- net UART_RX: track 0.00 -> 22.1 mm
- net UART_TX: track 0.00 -> 22.1 mm
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- added copper zone on F.Cu, net GND
Other:
- board size 120 x 63 mm -> 120 x 66 mm
- board text added: "SP4 breakout above (11 mm)"

Commit message: Carrier rev C (simple): checkpoint-3 fixes (P4KE10A TVS per panel lead, wire-loop test points), board 120 x 68 mm, build guide and shopping list
- D12-D16 P4KE10A (DO-41 standing) at the panel-lead connectors; TP2/TP3/TP4 low wire loops (TP2/TP4 under the breakout)
- J13 UART order kept as rev A/B (1 GND, 2 TX, 3 RX); ui.py docstring fixed
- layout: TVS rows, R56/CSN lowered, board 66 -> 68 mm so the GND pour keeps a >= 1.9 mm channel between its halves
- own 3D stand-in for the 3.81 mm vertical DO-41 (none upstream); ERC 0/0, DRC 0/0/0, 4 wire links, renders resolved
- hw/REVC_GUIDE.md, hw/REVC_SHOPPING.md, DESIGN_NOTES rev C section, BoM EUR 145.51/box; reviewer fixes in the guide

Co-Authored-By: Claude Opus 5.5 <noreply@anthropic.com>
Claude-Session: https://claude.ai/code/session_01PKzvcoWGaf5niy6TrXYsya
Parts:
- added D12: P4KE10A TVS, Diode_THT:D_DO-41_SOD81_P3.81mm_Vertical_CathodeUp, B.Cu at (134.2, 109.6)
- added D13: P4KE10A TVS, Diode_THT:D_DO-41_SOD81_P3.81mm_Vertical_CathodeUp, B.Cu at (142.7, 109.6)
- added D14: P4KE10A TVS, Diode_THT:D_DO-41_SOD81_P3.81mm_Vertical_CathodeUp, B.Cu at (107.0, 54.0)
- added D15: P4KE10A TVS, Diode_THT:D_DO-41_SOD81_P3.81mm_Vertical_CathodeUp, B.Cu at (92.5, 54.0)
- added D16: P4KE10A TVS, Diode_THT:D_DO-41_SOD81_P3.81mm_Vertical_CathodeUp, B.Cu at (158.7, 102.3)
- TP2, TP3, TP4: footprint TestPoint:TestPoint_Keystone_5010-5014_Multipurpose -> TestPoint:TestPoint_Loop_D2.50mm_Drill1.0mm
- moved R56 3.35 mm to (107.7, 57.1)
- moved MH2 2.00 mm to (166.5, 114.5)
- moved R54 1.20 mm to (139.9, 113.0)
- moved R55 1.20 mm to (142.2, 113.0)
- moved J10 0.60 mm to (134.2, 105.0)
- moved J11 0.60 mm to (142.7, 105.0)
- moved J23 0.60 mm to (151.2, 105.0)
Routing:
- net SW_MODE_NM: track 17.9 -> 14.6 mm
- net /ui/SW_MODE_MRM_J: track 15.1 -> 17.3 mm
- net /ui/SW_MODE_NM_J: track 5.78 -> 7.97 mm
- net /power/PWR_SW_J: track 8.71 -> 10.6 mm
- net /ui/SW_ROLE_J: track 6.41 -> 8.21 mm
- net /ui/BTN_TXRX_J: track 11.9 -> 13.7 mm
- net SW_ROLE: track 73.6 -> 74.8 mm
- net BTN_TXRX: track 50.8 -> 52.0 mm
Other:
- board size 120 x 66 mm -> 120 x 68 mm

Commit message: Rev C: TP2 away from the breakout's downward J2 pins; 'no J2 on box breakouts' in guide + drawing
The SP4 breakout's own 1x2 bench header J2 points down and its pins end ~2.5 mm
above the carrier, right over TP2 (5 V loop): one touch put 5 V on the radio's
3.3 V. TP2 moved below C11 (>= 3.7 mm from the J2 pins, no copper within 2 mm),
the 5 V stub shortened; guide (sections 2, 4E, common mistakes) and the placement
drawing say not to fit J2 on box breakouts. DRC 0/0/0, 4 links, BoM unchanged.

Co-Authored-By: Claude Opus 5.5 <noreply@anthropic.com>
Claude-Session: https://claude.ai/code/session_01PKzvcoWGaf5niy6TrXYsya
Parts:
- moved TP2 3.62 mm to (57.5, 74.5)
Routing:
- net 5V_PI: track 149.4 -> 147.4 mm
